Commit message: fix: wrap Gazebo plugins in xacro macro

File: src/a300_description/urdf/a300.gazebo.xacro (robot description, xacro)
@@ -1,6 +1,6 @@
 <?xml version="1.0"?>
-<robot xmlns:xacro="http://www.ros.org/wiki/xacro" name="a300_gazebo">
+<robot xmlns:xacro="http://www.ros.org/wiki/xacro" name="a300_gazebo"><xacro:macro name="a300_gazebo_plugins">
   <xacro:macro name="a300_gazebo_plugins" params="">
     <!-- Gazebo-specific systems will be added after the measured wheel geometry is available. -->
   </xacro:macro>
-</robot>
+</xacro:macro></robot>

Commit message: feat: complete Gazebo simulation stack

File: src/a300_description/urdf/a300.gazebo.xacro (robot description, xacro)
@@ -1,6 +1,36 @@
 <?xml version="1.0"?>
-<robot xmlns:xacro="http://www.ros.org/wiki/xacro" name="a300_gazebo"><xacro:macro name="a300_gazebo_plugins">
-  <xacro:macro name="a300_gazebo_plugins" params="">
-    <!-- Gazebo-specific systems will be added after the measured wheel geometry is available. -->
+<robot xmlns:xacro="http://www.ros.org/wiki/xacro" name="a300_gazebo">
+  <xacro:macro name="a300_gazebo_plugins">
+    <gazebo reference="left_wheel"><mu1>1.2</mu1><mu2>1.2</mu2></gazebo>
+    <gazebo reference="right_wheel"><mu1>1.2</mu1><mu2>1.2</mu2></gazebo>
+    <gazebo reference="caster"><mu1>0.2</mu1><mu2>0.2</mu2></gazebo>
+    <gazebo>
+      <plugin filename="gz-sim-diff-drive-system" name="gz::sim::systems::DiffDrive">
+        <left_joint>left_wheel_joint</left_joint><right_joint>right_wheel_joint</right_joint>
+        <wheel_separation>0.55</wheel_separation><wheel_radius>0.18</wheel_radius>
+        <max_linear_velocity>0.80</max_linear_velocity><min_linear_velocity>-0.80</min_linear_velocity>
+        <max_angular_velocity>1.00</max_angular_velocity><min_angular_velocity>-1.00</min_angular_velocity>
+        <max_linear_acceleration>1.0</max_linear_acceleration><min_linear_acceleration>-1.0</min_linear_acceleration>
+        <max_angular_acceleration>2.0</max_angular_acceleration><min_angular_acceleration>-2.0</min_angular_acceleration>
+        <topic>/cmd_vel</topic><odom_topic>/odom</odom_topic><tf_topic>/tf</tf_topic>
+        <frame_id>odom</frame_id><child_frame_id>base_link</child_frame_id><odom_publish_frequency>50</odom_publish_frequency>
+      </plugin>
+      <plugin filename="gz-sim-joint-state-publisher-system" name="gz::sim::systems::JointStatePublisher">
+        <topic>/joint_states</topic><joint_name>left_wheel_joint</joint_name><joint_name>right_wheel_joint</joint_name><update_rate>50</update_rate>
+      </plugin>
+    </gazebo>
+    <gazebo reference="laser_link">
+      <sensor name="r5_lidar" type="gpu_lidar">
+        <always_on>true</always_on><visualize>true</visualize><update_rate>10</update_rate>
+        <topic>/scan</topic><gz_frame_id>laser_link</gz_frame_id>
+        <lidar>
+          <scan>
+            <horizontal><samples>400</samples><resolution>1</resolution><min_angle>-3.14159265359</min_angle><max_angle>3.14159265359</max_angle></horizontal>
+            <vertical><samples>1</samples><resolution>1</resolution><min_angle>0</min_angle><max_angle>0</max_angle></vertical>
+          </scan>
+          <range><min>0.05</min><max>12.0</max><resolution>0.01</resolution></range>
+        </lidar>
+      </sensor>
+    </gazebo>
   </xacro:macro>
-</xacro:macro></robot>
+</robot>
