Commit message: feat: complete Gazebo simulation stack

File: src/a300_description/urdf/a300.urdf.xacro (robot description, xacro)
@@ -1,13 +1,23 @@
 <?xml version="1.0"?>
 <robot xmlns:xacro="http://www.ros.org/wiki/xacro" name="a300">
-<xacro:property name="body_length" value="0.75"/><xacro:property name="body_width" value="0.62"/><xacro:property name="body_height" value="0.75"/><xacro:property name="wheel_radius" value="0.18"/><xacro:property name="wheel_width" value="0.05"/><xacro:property name="wheel_track" value="0.55"/><xacro:property name="lidar_height" value="0.70"/>
-<material name="body"><color rgba="0.2 0.2 0.2 1"/></material><material name="wheel"><color rgba="0.05 0.05 0.05 1"/></material>
-<link name="base_link"><visual><origin xyz="0 0 0.40"/><geometry><box size="${body_length} ${body_width} ${body_height}"/></geometry><material name="body"/></visual><collision><origin xyz="0 0 0.40"/><geometry><box size="${body_length} ${body_width} ${body_height}"/></geometry></collision><inertial><origin xyz="0 0 0.40"/><mass value="60"/><inertia ixx="3" ixy="0" ixz="0" iyy="4" iyz="0" izz="4"/></inertial></link>
-<link name="left_wheel"><visual><geometry><cylinder radius="${wheel_radius}" length="${wheel_width}"/></geometry><material name="wheel"/></visual><collision><geometry><cylinder radius="${wheel_radius}" length="${wheel_width}"/></geometry></collision></link>
-<link name="right_wheel"><visual><geometry><cylinder radius="${wheel_radius}" length="${wheel_width}"/></geometry><material name="wheel"/></visual><collision><geometry><cylinder radius="${wheel_radius}" length="${wheel_width}"/></geometry></collision></link>
-<joint name="left_wheel_joint" type="continuous"><parent link="base_link"/><child link="left_wheel"/><origin xyz="0 ${wheel_track/2} ${wheel_radius}" rpy="1.5708 0 0"/><axis xyz="0 0 1"/></joint>
-<joint name="right_wheel_joint" type="continuous"><parent link="base_link"/><child link="right_wheel"/><origin xyz="0 -${wheel_track/2} ${wheel_radius}" rpy="1.5708 0 0"/><axis xyz="0 0 1"/></joint>
-<link name="caster"><visual><origin xyz="0 0 0.08"/><geometry><sphere radius="0.08"/></geometry></visual><collision><origin xyz="0 0 0.08"/><geometry><sphere radius="0.08"/></geometry></collision></link>
-<joint name="caster_joint" type="fixed"><parent link="base_link"/><child link="caster"/><origin xyz="-0.28 0 0"/></joint>
-<link name="laser_link"/><joint name="laser_joint" type="fixed"><parent link="base_link"/><child link="laser_link"/><origin xyz="0.20 0 ${lidar_height}"/></joint>
+  <xacro:arg name="use_sim" default="false"/>
+  <material name="body"><color rgba="0.2 0.2 0.2 1"/></material>
+  <material name="wheel"><color rgba="0.05 0.05 0.05 1"/></material>
+  <link name="base_link">
+    <visual><origin xyz="0 0 0.40"/><geometry><box size="0.75 0.62 0.75"/></geometry><material name="body"/></visual>
+    <collision><origin xyz="0 0 0.40"/><geometry><box size="0.75 0.62 0.75"/></geometry></collision>
+    <inertial><origin xyz="0 0 0.40"/><mass value="60"/><inertia ixx="3.0" ixy="0" ixz="0" iyy="4.0" iyz="0" izz="4.0"/></inertial>
+  </link>
+  <link name="left_wheel"><visual><geometry><cylinder radius="0.18" length="0.05"/></geometry><material name="wheel"/></visual><collision><geometry><cylinder radius="0.18" length="0.05"/></geometry></collision><inertial><mass value="2.0"/><inertia ixx="0.03" ixy="0" ixz="0" iyy="0.03" iyz="0" izz="0.03"/></inertial></link>
+  <link name="right_wheel"><visual><geometry><cylinder radius="0.18" length="0.05"/></geometry><material name="wheel"/></visual><collision><geometry><cylinder radius="0.18" length="0.05"/></geometry></collision><inertial><mass value="2.0"/><inertia ixx="0.03" ixy="0" ixz="0" iyy="0.03" iyz="0" izz="0.03"/></inertial></link>
+  <joint name="left_wheel_joint" type="continuous"><parent link="base_link"/><child link="left_wheel"/><origin xyz="0 0.275 0.18" rpy="1.5708 0 0"/><axis xyz="0 0 1"/></joint>
+  <joint name="right_wheel_joint" type="continuous"><parent link="base_link"/><child link="right_wheel"/><origin xyz="0 -0.275 0.18" rpy="1.5708 0 0"/><axis xyz="0 0 1"/></joint>
+  <link name="caster"><visual><origin xyz="0 0 0.08"/><geometry><sphere radius="0.08"/></geometry></visual><collision><origin xyz="0 0 0.08"/><geometry><sphere radius="0.08"/></geometry></collision><inertial><mass value="1.0"/><inertia ixx="0.003" ixy="0" ixz="0" iyy="0.003" iyz="0" izz="0.003"/></inertial></link>
+  <joint name="caster_joint" type="fixed"><parent link="base_link"/><child link="caster"/><origin xyz="-0.28 0 0"/></joint>
+  <link name="laser_link"><visual><geometry><cylinder radius="0.025" length="0.04"/></geometry></visual><inertial><mass value="0.2"/><inertia ixx="0.0001" ixy="0" ixz="0" iyy="0.0001" iyz="0" izz="0.0001"/></inertial></link>
+  <joint name="laser_joint" type="fixed"><parent link="base_link"/><child link="laser_link"/><origin xyz="0.20 0 0.70"/></joint>
+  <xacro:if value="$(arg use_sim)">
+    <xacro:include filename="$(find a300_description)/urdf/a300.gazebo.xacro"/>
+    <xacro:a300_gazebo_plugins/>
+  </xacro:if>
 </robot>

Commit message: 可验证版，初步实现了自动刹车

File: src/a300_description/urdf/a300.urdf.xacro (robot description, xacro)
@@ -16,5 +16,5 @@
   <joint name="caster_joint" type="fixed"><parent link="base_link"/><child link="caster"/><origin xyz="-0.28 0 0"/></joint>
   <link name="laser_link"><visual><geometry><cylinder radius="0.025" length="0.04"/></geometry></visual><inertial><mass value="0.2"/><inertia ixx="0.0001" ixy="0" ixz="0" iyy="0.0001" iyz="0" izz="0.0001"/></inertial></link>
-  <joint name="laser_joint" type="fixed"><parent link="base_link"/><child link="laser_link"/><origin xyz="0.20 0 0.70"/></joint>
+  <joint name="laser_joint" type="fixed"><parent link="base_link"/><child link="laser_link"/><origin xyz="0.20 0 0.85"/></joint>
   <xacro:if value="$(arg use_sim)">
     <xacro:include filename="$(find a300_description)/urdf/a300.gazebo.xacro"/>
